Commit message: setup

File: robot/robot_description.urdf (robot description, URDF)
Before this commit: robot visual, 10 links, 9 joints
Links:
- link base_link: geometry collision mesh filename=file:///home/samee/modulARM_sim/robot/base_link.stl scale=0.1 0.1 0.1; visual mesh filename=file:///home/samee/modulARM_sim/robot/base_link.stl scale=0.1 0.1 0.1
- link clamp: geometry collision mesh filename=file:///home/samee/modulARM_sim/robot/clamp.stl scale=0.1 0.1 0.1; visual mesh filename=file:///home/samee/modulARM_sim/robot/clamp.stl scale=0.1 0.1 0.1
- link clamp2: geometry collision mesh filename=file:///home/samee/modulARM_sim/robot/clamptop.stl scale=0.1 0.1 0.1; visual mesh filename=file:///home/samee/modulARM_sim/robot/clamptop.stl scale=0.1 0.1 0.1
- link clampEE: geometry collision mesh filename=file:///home/samee/modulARM_sim/robot/clampEE.stl scale=0.1 0.1 0.1; visual mesh filename=file:///home/samee/modulARM_sim/robot/clampEE.stl scale=0.1 0.1 0.1
- link clampb2: geometry collision mesh filename=file:///home/samee/modulARM_sim/robot/clamp.stl scale=0.1 0.1 0.1; visual mesh filename=file:///home/samee/modulARM_sim/robot/clamp.stl scale=0.1 0.1 0.1
- link link: geometry collision mesh filename=file:///home/samee/modulARM_sim/robot/link.stl scale=0.1 0.1 0.1; visual mesh filename=file:///home/samee/modulARM_sim/robot/link.stl scale=0.1 0.1 0.1
- link link2: geometry collision mesh filename=file:///home/samee/modulARM_sim/robot/link.stl scale=0.1 0.1 0.1; visual mesh filename=file:///home/samee/modulARM_sim/robot/link.stl scale=0.1 0.1 0.1
- link shaft: geometry collision mesh filename=file:///home/samee/modulARM_sim/robot/shaft.stl scale=0.1 0.1 0.1; visual mesh filename=file:///home/samee/modulARM_sim/robot/shaft.stl scale=0.1 0.1 0.1
- link shaft2: geometry collision mesh filename=file:///home/samee/modulARM_sim/robot/shaft.stl scale=0.1 0.1 0.1; visual mesh filename=file:///home/samee/modulARM_sim/robot/shaft.stl scale=0.1 0.1 0.1
Joints:
- joint joint2: limit lower=-1.0 upper=1.0 effort=100 velocity=100 -> lower=-0.5 upper=0.5 effort=100 velocity=100
- joint jointEE: limit lower=-1.0 upper=1.0 effort=100 velocity=100 -> lower=-0.5 upper=0.5 effort=100 velocity=100
- joint joint_link: limit lower=-1.0 upper=1.0 effort=100 velocity=100 -> lower=-0.5 upper=0.5 effort=100 velocity=100
- joint joint_link2: limit lower=-1.0 upper=1.0 effort=100 velocity=100 -> lower=-0.5 upper=0.5 effort=100 velocity=100
- joint joint_shaft: limit lower=-1.0 upper=1.0 effort=100 velocity=100 -> lower=-0.5 upper=0.5 effort=100 velocity=100
- joint joint_shaft2: limit lower=-1.0 upper=1.0 effort=100 velocity=100 -> lower=-0.5 upper=0.5 effort=100 velocity=100
- joint shaft_joint: limit lower=-1.0 upper=1.0 effort=100 velocity=100 -> lower=-0.5 upper=0.5 effort=100 velocity=100
- joint shaft_joint2: limit lower=-1.0 upper=1.0 effort=100 velocity=100 -> lower=-0.5 upper=0.5 effort=100 velocity=100
